File: flat_memory_8k.kicad_sch (KiCad schematic)
At the start: 34 parts, among them X1 Power, X2 Address, X3 Data, X4 Mode, X5 Control, X6 Clock

Commit message: Add files via upload
Add optional footprint for memory
Добавлены опциональные посадочные места памяти
Parts:
- added C19, C21, C23: 100n, Capacitor_SMD:C_0805_2012Metric_Pad1.18x1.45mm_HandSolder, symbol Device:C
- added C20, C22, C24: 1u, Capacitor_Tantalum_SMD:CP_EIA-3216-18_Kemet-A_Pad1.58x1.35mm_HandSolder, symbol Device:C_Polarized
- added DD10: DUAL SOCKET, Package_DIP:DIP-24_W7.62mm_LongPads, symbol К580-К1810-К1821:CAT28C16A
- added DD11, DD12: DUAL SOCKET, Package_DIP:DIP-24_W7.62mm_LongPads, symbol К580-К1810-К1821:537РУ10
- added JP1: Jumper_2_Open, Jumper:SolderJumper-2_P1.3mm_Open_RoundedPad1.0x1.5mm, symbol Jumper:Jumper_2_Open
Connections:
- net +5: now also C19.1, C20.1, C21.1, C22.1, C23.1, C24.1, DD10.24 (VCC), DD11.24 (VCC), DD12.24 (VCC)
- net AB0: now also DD10.8 (A0), DD11.8 (A10), DD12.8 (A10)
- net AB1: now also DD10.7 (A1), DD11.7 (A9), DD12.7 (A9)
- net AB10: now also DD10.19 (A10), DD11.19 (A0), DD12.19 (A0)
- net AB2: now also DD10.6 (A2), DD11.6 (A8), DD12.6 (A8)
- net AB3: now also DD10.5 (A3), DD11.5 (A7), DD12.5 (A7)
- net AB4: now also DD10.4 (A4), DD11.4 (A6), DD12.4 (A6)
- net AB5: now also DD10.3 (A5), DD11.3 (A5), DD12.3 (A5)
- net AB6: now also DD10.2 (A6), DD11.2 (A4), DD12.2 (A4)
- net AB7: now also DD10.1 (A7), DD11.1 (A3), DD12.1 (A3)
- net AB8: now also DD10.23 (A8), DD11.23 (A2), DD12.23 (A2)
- net AB9: now also DD10.22 (A9), DD11.22 (A1), DD12.22 (A1)
- net DATA_B0: now also DD10.9 (Q0), DD11.9 (Q0), DD12.9 (Q0)
- net DATA_B1: now also DD10.10 (Q1), DD11.10 (Q1), DD12.10 (Q1)
- net DATA_B2: now also DD10.11 (Q2), DD11.11 (Q2), DD12.11 (Q2)
- net DATA_B3: now also DD10.13 (Q3), DD11.13 (Q3), DD12.13 (Q3)
- net DATA_B4: now also DD10.14 (Q4), DD11.14 (Q4), DD12.14 (Q4)
- net DATA_B5: now also DD10.15 (Q5), DD11.15 (Q5), DD12.15 (Q5)
- net DATA_B6: now also DD10.16 (Q6), DD11.16 (Q6), DD12.16 (Q6)
- net DATA_B7: now also DD10.17 (Q7), DD11.17 (Q7), DD12.17 (Q7)
- net GND: now also C19.2, C20.2, C21.2, C22.2, C23.2, C24.2, DD10.12 (GND), DD11.12 (GND), DD12.12 (GND)
- net ~{4K_CS}: now also DD10.18 (~{CE})
- net ~{6K_CS}: now also DD11.18 (~{CE})
- net ~{8K_CS}: now also DD12.18 (~{CE})
- net ~{MEMR}: now also DD10.20 (~{OE}), DD11.20 (~{OE}), DD12.20 (~{OE})
- net ~{MEMW}: now also DD10.21 (~{WE}), DD11.21 (~{WE}), DD12.21 (~{WE}), JP1.2 (B)
- net at DD1.21 (Vpp): now also JP1.1 (A)
- no-connect marks 12 -> 11

Commit message: Update
Parts:
- added C13: 100n, Capacitor_SMD:C_0805_2012Metric_Pad1.18x1.45mm_HandSolder, symbol Device:C
- renumbered C13 to C14, C14 to C15, C15 to C16, C16 to C17, C17 to C18, C18 to C19, C19 to C20, C20 to C21, C21 to C22, C22 to C23, C23 to C24, C24 to C25
Connections:
- net GND: now also C13.1
- net at DD9.6 (E3), R1.1: now also C13.2
- net INTE renamed ~{WRQ}
- net Single_BCLK renamed F2TTL
- net Single_OSC_TTL renamed OSC_TTL
Other:
- moved on the sheet: R1
